File: WakeOnWifi.sch (EAGLE design)
At the start: 7 parts

Commit message: WakeOnWifi board fixes
Parts:
- removed VIN: (no value), pinhead:PINHD-1X2
- added SOFTWARE: (no value), pinhead:PINHD-1X2
Connections:
- removed net +5V: VIN.1
- removed net GND: VIN.2
- new net N$6: ARDUINORIGHT.10, SOFTWARE.1
- new net N$7: ARDUINORIGHT.9, SOFTWARE.2
Changed lines of the file:
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@@
 <setting verticaltext="up"/>
 </settings>
-<grid distance="0.1" unitdist="inch" unit="inch" style="lines" multiple="1" display="yes" altdistance="0.01" altunitdist="inch" altunit="inch"/>
+<grid distance="0.1" unitdist="inch" unit="inch" style="lines" multiple="1" display="no" altdistance="0.01" altunitdist="inch" altunit="inch"/>
 <layers>
 <layer number="1" name="Top" color="4" fill="1" visible="no" active="no"/>
@@
 <part name="WIFI" library="con-lstb" deviceset="MA04-2" device=""/>
 <part name="VOUT" library="pinhead" deviceset="PINHD-1X2" device=""/>
-<part name="VIN" library="pinhead" deviceset="PINHD-1X2" device=""/>
-<part name="P+1" library="supply1" deviceset="+5V" device=""/>
-<part name="GND1" library="supply1" deviceset="GND" device=""/>
 <part name="RELAY" library="pinhead" deviceset="PINHD-1X3" device=""/>
 <part name="RS232" library="pinhead" deviceset="PINHD-1X2" device=""/>
+<part name="SOFTWARE" library="pinhead" deviceset="PINHD-1X2" device=""/>
 </parts>
 <sheets>
@@
 </instance>
 <instance part="VOUT" gate="G$1" x="91.44" y="10.16"/>
-<instance part="VIN" gate="G$1" x="114.3" y="10.16"/>
-<instance part="P+1" gate="1" x="129.54" y="30.48"/>
-<instance part="GND1" gate="1" x="129.54" y="2.54"/>
 <instance part="RELAY" gate="A" x="129.54" y="68.58"/>
 <instance part="RS232" gate="G$1" x="33.02" y="58.42" rot="R180"/>
+<instance part="SOFTWARE" gate="G$1" x="93.98" y="55.88"/>
 </instances>
 <busses>
 </busses>
 <nets>
-<net name="GND" class="0">
-<segment>
-<pinref part="VIN" gate="G$1" pin="2"/>
-<pinref part="GND1" gate="1" pin="GND"/>
-<wire x1="111.76" y1="10.16" x2="111.76" y2="0" width="0.1524" layer="91"/>
-<wire x1="111.76" y1="0" x2="119.38" y2="0" width="0.1524" layer="91"/>
-<wire x1="119.38" y1="0" x2="119.38" y2="10.16" width="0.1524" layer="91"/>
-<wire x1="119.38" y1="10.16" x2="129.54" y2="10.16" width="0.1524" layer="91"/>
-<wire x1="129.54" y1="10.16" x2="129.54" y2="5.08" width="0.1524" layer="91"/>
-</segment>
-</net>
-<net name="+5V" class="0">
-<segment>
-<pinref part="VIN" gate="G$1" pin="1"/>
-<wire x1="129.54" y1="27.94" x2="129.54" y2="20.32" width="0.1524" layer="91"/>
-<wire x1="129.54" y1="20.32" x2="111.76" y2="20.32" width="0.1524" layer="91"/>
-<wire x1="111.76" y1="20.32" x2="111.76" y2="12.7" width="0.1524" layer="91"/>
-<pinref part="P+1" gate="1" pin="+5V"/>
-</segment>
-</net>
 <net name="N$1" class="0">
 <segment>
@@
 </segment>
 </net>
+<net name="N$6" class="0">
+<segment>
+<pinref part="ARDUINORIGHT" gate="1" pin="10"/>
+<pinref part="SOFTWARE" gate="G$1" pin="1"/>
+<wire x1="81.28" y1="58.42" x2="91.44" y2="58.42" width="0.1524" layer="91"/>
+</segment>
+</net>
+<net name="N$7" class="0">
+<segment>
+<pinref part="ARDUINORIGHT" gate="1" pin="9"/>
+<pinref part="SOFTWARE" gate="G$1" pin="2"/>
+<wire x1="81.28" y1="55.88" x2="91.44" y2="55.88" width="0.1524" layer="91"/>
+</segment>
+</net>
